Commit message: now gripper is also working

File: move_it_config/config/arm.ros2_control.xacro (robot description, xacro)
@@ -57,4 +57,44 @@
                 <state_interface name="velocity"/>
             </joint>
+            <joint name="left_inner_knuckle_joint">
+              <command_interface name="position"/>
+              <state_interface name="position"/>
+              <state_interface name="velocity"/>
+              <param name="mimic">finger_joint</param>
+              <param name="multiplier">1.0</param>
+              <param name="offset">0.0</param>
+            </joint>
+            <joint name="left_inner_finger_joint">
+              <command_interface name="position"/>
+              <state_interface name="position"/>
+              <state_interface name="velocity"/>
+              <param name="mimic">finger_joint</param>
+              <param name="multiplier">1.0</param>
+              <param name="offset">0.0</param>
+            </joint>
+            <joint name="right_inner_knuckle_joint">
+              <command_interface name="position"/>
+              <state_interface name="position"/>
+              <state_interface name="velocity"/>
+              <param name="mimic">finger_joint</param>
+              <param name="multiplier">-1.0</param>
+              <param name="offset">0.0</param>
+            </joint>
+            <joint name="right_inner_finger_joint">
+              <command_interface name="position"/>
+              <state_interface name="position"/>
+              <state_interface name="velocity"/>
+              <param name="mimic">finger_joint</param>
+              <param name="multiplier">-1.0</param>
+              <param name="offset">0.0</param>
+            </joint>
+            <joint name="right_outer_knuckle_joint">
+              <command_interface name="position"/>
+              <state_interface name="position"/>
+              <state_interface name="velocity"/>
+              <param name="mimic">finger_joint</param>
+              <param name="multiplier">-1.0</param>
+              <param name="offset">0.0</param>
+            </joint>
         </ros2_control>
     </xacro:macro>
